File: KiCad_Curve_Tracer_PCB/KiCad_Curve_Tracer_PCB.kicad_pcb (KiCad board)
At the start: 2 copper layers, 21.6 x 31.7 mm, 9 parts, among them J1 Vi, J2 DUT, J3 rng, J4 Input, U1 Opamp_Dual

Commit message: added 3 PCB projects
Parts:
- added G***: LOGO, graphics:duck, B.Cu at (53.3, 36.1)
- added J5: Vo, Connector_PinHeader_2.54mm:PinHeader_1x02_P2.54mm_Vertical, F.Cu at (61.0, 58.4)
- C1, C2: footprint Capacitor_THT:C_Axial_L5.1mm_D3.1mm_P10.00mm_Horizontal -> Capacitor_THT:C_Disc_D3.0mm_W1.6mm_P2.50mm
- moved J3 12.7 mm to (50.7, 52.7)
- moved C1 5.46 mm to (61.2, 46.5)
- moved R2 2.43 mm to (54.2, 51.5)
- moved R1 1.04 mm to (57.3, 61.7)
- moved J2 1.04 mm to (61.0, 35.6)
- moved C2 0.37 mm to (46.3, 41.4)
- moved U1 0.18 mm to (49.9, 47.7)
Routing:
- net /opamp curve tracer/Vo: track 13.5 -> 25.8 mm
- net /opamp curve tracer/V+: track 25.6 -> 29.0 mm
- net /opamp curve tracer/DUT+: track 9.59 -> 12.0 mm
- net /opamp curve tracer/DUT-: track 20.6 -> 22.9 mm
- net /opamp curve tracer/rng: track 10.4 -> 11.0 mm
Other:
- board size 21.6 x 31.7 mm -> 20.3 x 31.7 mm
- board text added: "+"
- board text added: "-"
- board text added: "0.1u"
- board text added: "100"
- board text added: "100K"
- board text added: "DUT"
- board text added: "G"
- board text added: "Lee Evans"
- board text added: "POW"
- board text added: "TL052CP"
- board text added: "V1"
- board text added: "Vo"

Commit message: finished first draft of all 3
Parts:
- moved J4 5.08 mm to (45.7, 50.8)
- moved J3 0.68 mm to (50.7, 53.3)
Routing:
- net /opamp curve tracer/V-: track 19.7 -> 14.6 mm
- net /opamp curve tracer/rng: track 11.0 -> 10.4 mm
Other:
- board text added: "Vi"
- board text added: "rng"
- board text removed: "Lee Evans"
- board text removed: "V1"
Changed lines of the file:
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@@
 	(footprint "Connector_PinHeader_2.54mm:PinHeader_1x03_P2.54mm_Vertical"
 		(layer "F.Cu")
-		(at 45.72 55.88)
+		(at 45.72 50.8)
 		(descr "Through hole straight pin header, 1x03, 2.54mm pitch, single row")
 		(tags "Through hole pin header THT 1x03 2.54mm single row")
@@
 	(footprint "Connector_PinHeader_2.54mm:PinHeader_1x02_P2.54mm_Vertical"
 		(layer "F.Cu")
-		(at 50.681593 52.664423)
+		(at 50.681593 53.34)
 		(descr "Through hole straight pin header, 1x02, 2.54mm pitch, single row")
 		(tags "Through hole pin header THT 1x02 2.54mm single row")
@@
 		(layer "Edge.Cuts")
 	)
-	(gr_text "Lee\nEvans"
-		(at 53.848 45.212 0)
-		(layer "B.Cu" knockout)
-		(effects
-			(font
-				(size 1 1)
-				(thickness 0.25)
-				(bold yes)
-			)
-			(justify bottom mirror)
-		)
-	)
 	(gr_text "100K"
 		(at 57.404 57.15 90)
@@
 		(effects
 			(font
-				(size 0.8 0.8)
+				(size 1 1)
 				(thickness 0.15)
 			)
@@
 	)
 	(gr_text "POW"
-		(at 44.18 63.754 0)
+		(at 44.077089 59.05772 0)
 		(layer "F.SilkS")
 		(effects
@@
 		(effects
 			(font
-				(size 0.8 0.8)
+				(size 1 1)
 				(thickness 0.15)
 			)
@@
 	)
 	(gr_text "Vo"
-		(at 60.452 55.118 270)
+		(at 60.452 54.61 270)
 		(layer "F.SilkS")
 		(effects
@@
 		(effects
 			(font
-				(size 0.8 0.8)
+				(size 1 1)
 				(thickness 0.15)
 			)
@@
 		(effects
 			(font
-				(size 0.8 0.8)
+				(size 1 1)
 				(thickness 0.15)
 			)
@@
 	)
 	(gr_text "G"
-		(at 47.498 57.658 270)
+		(at 47.357684 52.716884 270)
 		(layer "F.SilkS")
 		(effects
@@
 	)
 	(gr_text "+"
-		(at 47.498 60.198 270)
+		(at 47.416531 55.17806 270)
 		(layer "F.SilkS")
 		(effects
@@
 	)
 	(gr_text "-"
-		(at 47.498 55.02 270)
+		(at 47.475377 50.049168 270)
 		(layer "F.SilkS")
 		(effects
@@
 		)
 	)
+	(gr_text "rng"
+		(at 50.8 50.8 0)
+		(layer "F.SilkS")
+		(effects
+			(font
+				(size 1 1)
+				(thickness 0.15)
+			)
+		)
+	)
 	(gr_text "+"
 		(at 57.912 34.798 270)
@@
 		(effects
 			(font
-				(size 0.8 0.8)
+				(size 1 1)
 				(thickness 0.15)
 			)
 		)
 	)
-	(gr_text "V1"
+	(gr_text "Vi"
 		(at 47.68 37.084 270)
 		(layer "F.SilkS")
@@
 	)
 	(segment
-		(start 50.292 60.96)
-		(end 53.594 57.658)
+		(start 54.864 58.42)
+		(end 61.214 52.07)
 		(width 0.75)
 		(layer "B.Cu")
@@
 	)
 	(segment
-		(start 53.594 57.658)
-		(end 55.626 57.658)
+		(start 48.26 58.42)
+		(end 54.864 58.42)
 		(width 0.75)
 		(layer "B.Cu")
@@
 	)
 	(segment
-		(start 45.72 60.96)
-		(end 50.292 60.96)
+		(start 48.26 58.42)
+		(end 45.72 55.88)
 		(width 0.75)
 		(layer "B.Cu")
@@
 	)
 	(segment
-		(start 55.626 57.658)
-		(end 61.214 52.07)
-		(width 0.75)
-		(layer "B.Cu")
-		(net 2)
-	)
-	(segment
 		(start 46.31471 41.422)
 		(end 48.596785 41.422)
@@
 	)
 	(segment
-		(start 46.31471 41.422)
-		(end 44.704 43.03271)
+		(start 44.650523 43.086187)
+		(end 44.650523 49.730523)
+		(width 0.75)
+		(layer "F.Cu")
+		(net 3)
+	)
+	(segment
+		(start 44.650523 49.730523)
+		(end 45.72 50.8)
 		(width 0.75)
 		(layer "F.Cu")
@@
 	)
 	(segment
-		(start 44.704 43.03271)
-		(end 44.704 54.864)
-		(width 0.75)
-		(layer "F.Cu")
-		(net 3)
-	)
-	(segment
-		(start 44.704 54.864)
-		(end 45.72 55.88)
+		(start 46.31471 41.422)
+		(end 44.650523 43.086187)
 		(width 0.75)
 		(layer "F.Cu")
@@
 	)
 	(segment
-		(start 51.648423 52.664423)
-		(end 57.404 58.42)
+		(start 57.404 58.42)
+		(end 60.96 58.42)
 		(width 0.75)
 		(layer "F.Cu")
@@
 	)
 	(segment
-		(start 50.681593 52.664423)
-		(end 51.648423 52.664423)
-		(width 0.75)
-		(layer "F.Cu")
-		(net 7)
-	)
-	(segment
-		(start 57.404 58.42)
-		(end 60.96 58.42)
-		(width 0.75)
-		(layer "F.Cu")
-		(net 7)
-	)
-	(segment
 		(start 54.973415 49.131415)
 		(end 54.973415 47.74537)
@@
 	)
 	(segment
+		(start 52.324 53.34)
+		(end 57.404 58.42)
+		(width 0.75)
+		(layer "F.Cu")
+		(net 7)
+	)
+	(segment
+		(start 50.681593 53.34)
+		(end 52.324 53.34)
+		(width 0.75)
+		(layer "F.Cu")
+		(net 7)
+	)
+	(segment
 		(start 57.340842 54.800842)
 		(end 60.96 58.42)
@@
 	)
 	(segment
-		(start 50.681593 55.204423)
+		(start 50.681593 55.88)
 		(end 50.681593 58.130467)
 		(width 0.75)
@@
 		(polygon
 			(pts
-				(xy 43.18 33.02) (xy 64.77 33.02) (xy 64.77 64.77) (xy 43.18 64.77)
-			)
-		)
+				(xy 43.18 33.02) (xy 63.5 33.02) (xy 63.5 64.77) (xy 43.18 64.77)
+			)
+		)
